File: esquematico.kicad_pcb (KiCad board)
At the start: 2 copper layers, 46 parts, among them J1 Screw_Terminal_01x02, J11 valvula, J2 BORNERA 1, J3 BORNERA 1, J4 BORNERA 2, J5 BORNERA 2, J6 BORNERA 1, J7 BORNERA 2, J8 BORNERA 1, J9 BORNERA 2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

Commit message: terminamos el pcb falta ordenar un poco mas
Parts:
- moved R15 181.3 mm to (81.3, 177.0), turned to -90 degrees
- moved Q4 177.6 mm to (87.0, 176.0), turned to -90 degrees
- moved D4 166.9 mm to (108.0, 176.6)
- moved J1 165.5 mm to (52.7, 80.7), turned to -90 degrees
- moved U1 162.7 mm to (82.8, 123.2)
- moved R14 162.5 mm to (105.4, 168.3)
- moved U6 160.4 mm to (101.0, 162.0)
- moved R13 157.9 mm to (95.9, 161.0), turned to -90 degrees
- moved U2 156.3 mm to (61.0, 120.1), turned to 0 degrees
- moved R1 154.5 mm to (81.9, 120.7), turned to 0 degrees
- moved RL4 148.0 mm to (117.5, 179.1), turned to 0 degrees
- moved J9 125.5 mm to (142.2, 163.9), turned to 180 degrees
- moved J8 124.3 mm to (132.1, 186.8), turned to 0 degrees
- moved J2 112.6 mm to (132.8, 80.6), turned to 0 degrees
- moved J5 112.2 mm to (143.0, 54.0), turned to 180 degrees
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Connections:
- J4 pad 1: NC2.1 -> NO2.1
- J4 pad 3: NO2.1 -> NC2.1
- J5 pad 1: NC2 -> NO2
- J5 pad 3: NO2 -> NC2
- J7 pad 1: NC2.2 -> NO2.2
- J7 pad 3: NO2.2 -> NC2.2
- J9 pad 1: NC2.3 -> NO2.3
- J9 pad 3: NO2.3 -> NC2.3
- R1 pad 1: GPIO33 -> GPIO18
- R13 pad 1: GPIO32 -> GPIO17
- R5 pad 1: GPIO4 -> GPIO21
- R9 pad 1: GPIO15 -> GPIO19
- U2 pad J2-7: GPIO32 -> unconnected-(U2-IO32-PadJ2-7)
- U2 pad J2-8: GPIO33 -> unconnected-(U2-IO33-PadJ2-8)
- U2 pad J3-11: unconnected-(U2-IO17-PadJ3-11) -> GPIO17
- U2 pad J3-13: GPIO4 -> unconnected-(U2-IO4-PadJ3-13)
- U2 pad J3-16: GPIO15 -> unconnected-(U2-IO15-PadJ3-16)
- U2 pad J3-6: unconnected-(U2-IO21-PadJ3-6) -> GPIO21
- U2 pad J3-8: unconnected-(U2-IO19-PadJ3-8) -> GPIO19
- U2 pad J3-9: unconnected-(U2-IO18-PadJ3-9) -> GPIO18
Routing:
- net 12V: track 0.00 -> 356.5 mm, vias 0 -> 4
- net GPIO21: track 0.00 -> 73.0 mm, vias 0 -> 1
- net GPIO17: track 0.00 -> 61.6 mm, vias 0 -> 1
- net GPIO19: track 0.00 -> 42.9 mm, vias 0 -> 1
- net Net-(D4-A): track 0.00 -> 33.3 mm, vias 0 -> 2
- net Net-(D3-A): track 0.00 -> 27.9 mm, vias 0 -> 2
- net Net-(D1-A): track 0.00 -> 25.2 mm, vias 0 -> 2
- net Net-(Q4-G): track 0.00 -> 24.7 mm, vias 0 -> 1
- net Net-(D2-A): track 0.00 -> 22.7 mm, vias 0 -> 2
- net Net-(Q3-G): track 0.00 -> 18.9 mm, vias 0 -> 1
- net Net-(Q1-G): track 0.00 -> 18.2 mm, vias 0 -> 1
- net NO1.3: track 0.00 -> 15.8 mm
- net Net-(Q2-G): track 0.00 -> 13.5 mm, vias 0 -> 1
- net NC2: track 0.00 -> 10.4 mm
- net COM2: track 0.00 -> 10.4 mm
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- added copper zone on B.Cu, net GND
- added copper zone on F.Cu, net GND
